Commit message: add launch file

File: go1_description/xacro/robot.xacro (robot description, xacro)
@@ -24,9 +24,21 @@
     <link name="rslidar" />
     <joint name="rslidar_joint" type="fixed">
-      <origin rpy="0 0 0" xyz="0.1 0 0.07"/>
-      <parent link="base"/>
+      <origin rpy="0 0 0" xyz="0.1 0 0.13"/>
+      <parent link="base_link"/>
       <child link="rslidar"/>
     </joint>
-    <link name="base">
+    <link name="lidar" />
+    <joint name="lidar_joint" type="fixed">
+      <origin rpy="0 0 0" xyz="0.1 0 0.13"/>
+      <parent link="base_link"/>
+      <child link="lidar"/>
+    </joint>
+    <link name="velodyne" />
+    <joint name="velodyne_joint" type="fixed">
+      <origin rpy="0 0 0" xyz="0.1 0 0.13"/>
+      <parent link="base_link"/>
+      <child link="velodyne"/>
+    </joint>
+    <link name="base_link">
         <visual>
             <origin rpy="0 0 0" xyz="0 0 0"/>
@@ -38,5 +50,5 @@
     <joint name="floating_base" type="fixed">
         <origin rpy="0 0 0" xyz="0 0 0"/>
-        <parent link="base"/>
+        <parent link="base_link"/>
         <child link="trunk"/>
     </joint>

Commit message: fix imu bug

File: go1_description/xacro/robot.xacro (robot description, xacro)
@@ -79,5 +79,5 @@
         <parent link="trunk"/>
         <child link="imu_link"/>
-        <origin rpy="0 0 0" xyz="-0.01592 -0.06659 -0.00617"/>
+        <origin rpy="3.14 0 3.14" xyz="-0.01592 -0.06659 -0.00617"/>
     </joint>
     <link name="imu_link">
